File: HW/RSSI Detector.kicad_pcb (KiCad board)
At the start: 2 copper layers, 35.6 x 17.8 mm, 29 parts, among them P1 SMA, P2 SMA, U1 AD8319, U2 AD8319, U3 Teensy3.2, X1 CX3099NL

Commit message: fixed problems with 3d
Parts:
- removed the P1 at (0.00, 0.00)
